Commit message: successfully configurate the arm with sc

File: explorer_sc_arm_description/urdf/explorer_sc_arm_description.urdf (robot description, URDF)
Before this commit: robot explorer_sc_arm_description, 17 links, 16 joints
Links:
- link arm1_link: mass 0.740834240282329 -> 0.676426297298435
- link arm2_link: mass 0.432896616493016 -> 0.196076424497199
- link arm3_link: mass 0.251042694943515 -> 0.208381103991094
- link frame_link: mass 3.26161515055018 -> 1.7992512190132
- link left_down_wheel_link: mass 0.82612178476788 -> 0.0699947445973927
- link left_up_wheel_link: mass 0.826121794411708 -> 0.0699947504295786
- link right_down_wheel_link: mass 0.826121790600066 -> 0.0699947504295788
- link right_up_wheel_link: mass 0.826121794411715 -> 0.0699947504295802
Joints:
- joint left_down_wheel_base_joint: origin xyz=0.22551 0.28813 -0.091104 rpy=-7.0265E-33 1.1082E-16 -6.5165E-17 -> xyz=0.15861 0.28813 -0.091104 rpy=-7.0265E-33 1.1082E-16 -6.5165E-17
- joint left_up_wheel_base_joint: origin xyz=0.22551 -0.23931 -0.091104 rpy=-7.0265E-33 1.1082E-16 -6.5165E-17 -> xyz=0.15861 -0.23931 -0.091104 rpy=-3.9302E-35 0 0
- joint right_down_wheel_base_joint: origin xyz=-0.25469 0.28813 -0.091104 rpy=-7.0265E-33 1.1082E-16 -6.5165E-17 -> xyz=-0.16939 0.28813 -0.091104 rpy=-7.0265E-33 1.1082E-16 -6.5165E-17
- joint right_up_wheel_base_joint: origin xyz=-0.25469 -0.23931 -0.091104 rpy=-3.9302E-35 0 0 -> xyz=-0.16939 -0.23931 -0.091104 rpy=-3.9302E-35 0 0
- joint robot_left_right: axis 0 0 1 -> 0 0 0; limit effort=0 velocity=0 -> (none); origin xyz=0 0 0 rpy=-3.9302E-35 0 0 -> xyz=0 0 0 rpy=-3.93023761073179E-35 0 0; type revolute -> fixed
